File: Datalogger.kicad_pcb (KiCad board)
At the start: 4 copper layers, 55 x 30.3 mm, 55 parts, among them J1 MSD-1-A, J2 USB4216-03-A_REVA, Q1 NPN, Q2 NPN, U1 ESP32-C3-MINI-1-N4, U2 CP2102-GM, U3 BME280, U4 TLV76133DCYR

Commit message: finished 4 layer board
Parts:
- moved R2 24.8 mm to (226.5, 111.5), turned to 90 degrees
- moved C4 23.0 mm to (226.5, 110.0), turned to 0 degrees
- moved R3 19.4 mm to (221.5, 111.0), turned to 90 degrees
- moved C5 15.9 mm to (220.5, 109.0), turned to 180 degrees
- moved C8 14.0 mm to (205.0, 91.0), turned to 90 degrees
- moved C9 11.2 mm to (203.0, 91.0), turned to 90 degrees
- moved R17 6.45 mm to (195.5, 116.0), turned to 0 degrees
- moved D5 4.84 mm to (185.3, 89.0), turned to -90 degrees
- moved D1 4.68 mm to (187.2, 94.5), turned to 180 degrees
- moved R16 4.11 mm to (189.5, 111.5), turned to 0 degrees
- moved Q1 2.06 mm to (192.0, 113.5), turned to -90 degrees
- moved Q2 1.00 mm to (196.0, 113.0), turned to 90 degrees
- moved D3 1.00 mm to (188.0, 104.0)
- moved R5 0.91 mm to (185.8, 91.0), turned to 180 degrees
- moved C1 0.50 mm to (226.0, 92.5)
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Connections:
- H1 pad 1: unconnected-(H1-Pad1) -> GND
- H2 pad 1: unconnected-(H2-Pad1) -> GND
- H3 pad 1: unconnected-(H3-Pad1) -> GND
- H4 pad 1: unconnected-(H4-Pad1) -> GND
- R18 pad 1: /GPIO19 -> GPIO19
- R19 pad 1: /GPIO18 -> GPIO18
- U1 pad 26: /GPIO18 -> GPIO18
- U1 pad 27: /GPIO19 -> GPIO19
Routing:
- net GND: track 0.00 -> 144.8 mm, vias 0 -> 35
- net USB_DN: track 0.00 -> 65.1 mm
- net USB_DP: track 0.00 -> 58.2 mm, vias 0 -> 2
- net VCC_3V3: track 0.00 -> 53.1 mm, vias 0 -> 14
- net U0TXD: track 0.00 -> 50.9 mm, vias 0 -> 2
- net /CHIP_PU: track 0.00 -> 50.7 mm
- net U0RXD: track 0.00 -> 49.4 mm, vias 0 -> 2
- net /SPI_MISO: track 0.00 -> 31.2 mm, vias 0 -> 2
- net /GPIO09: track 0.00 -> 30.8 mm
- net RTS: track 0.00 -> 30.7 mm, vias 0 -> 2
- net /SPI_SCK: track 0.00 -> 28.2 mm
- net DTR: track 0.00 -> 24.9 mm, vias 0 -> 2
- net /SDA: track 0.00 -> 23.2 mm
- net /SPI_MOSI: track 0.00 -> 20.6 mm, vias 0 -> 2
- net VBUS: track 0.00 -> 18.1 mm, vias 0 -> 2
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- added copper zone on B.Cu, net GND
- added copper zone on F.Cu, net GND
- added copper zone on In1.Cu, net GND
- added copper zone on F.Cu, net VBUS
- added copper zone on F.Cu, net VCC_3V3
- added copper zone on In2.Cu, net VCC_3V3
