File: Datalogger.kicad_sch (KiCad schematic)
At the start: 31 parts, among them J1 MSD-1-A, Q1 NPN, Q2 NPN, U1 ESP32-C3-MINI-1-N4, U3 BME280

Commit message: finished 4 layer board
Connections:
- net GND: now also H1.1, H2.1, H3.1, H4.1
Other:
- moved on the sheet: R18, R19
